Commit message: ts materisl

File: urdf/materials.urdf.xacro (robot description, xacro)
@@ -6,5 +6,5 @@
 <robot xmlns:xacro="http://wiki.ros.org/xacro">
   <xacro:macro name="materials" params="tf_prefix">
-    <material name="${tf_prefix}black">
+    <material name="${tf_prefix}blackk">
       <color rgba="0.0 0.0 0.0 1.0"/>
     </material>

Commit message: ts material

File: urdf/materials.urdf.xacro (robot description, xacro)
@@ -6,5 +6,5 @@
 <robot xmlns:xacro="http://wiki.ros.org/xacro">
   <xacro:macro name="materials" params="tf_prefix">
-    <material name="${tf_prefix}blackk">
+    <material name="${tf_prefix}black">
       <color rgba="0.0 0.0 0.0 1.0"/>
     </material>
