Commit message: add tcp definition to gripper package

File: urdf/diy_gripper_model.urdf.xacro (robot description, xacro)
@@ -8,3 +8,10 @@
         <origin xyz="0 0 0" rpy="0 0 0"/>
     </xacro:diy_soft_gripper>
+    <!--add a TCP Link for convenience, show TCP reference set in rviz-->
+    <joint name="tcp_joint" type="fixed">
+        <origin xyz="0 0 0.08" rpy="0 0 0"/>
+        <parent link="$(arg tf_prefix)base_link"/>
+        <child link="$(arg tf_prefix)tcp_link"/>
+    </joint>
+    <link name="$(arg tf_prefix)tcp_link"/>
 </robot>
