Commit message: materials_troubleshooting

File: urdf/diy_gripper_macro.urdf.xacro (robot description, xacro)
@@ -18,5 +18,5 @@
           <mesh filename="package://diy_soft_gripper_description/meshes/visual/base_link.stl" scale="0.001 0.001 0.001"/>
         </geometry>
-        <material name="grey" />
+        <material name="${tf_prefix}grey" />
       </visual>
     <!--
@@ -41,5 +41,5 @@
           <mesh filename="package://diy_soft_gripper_description/meshes/visual/soft_finger.stl" scale="0.001 0.001 0.001"/>
         </geometry>
-        <material name="orange" />
+        <material name="${tf_prefix}orange" />
       </visual>
     <!--
@@ -64,5 +64,5 @@
           <mesh filename="package://diy_soft_gripper_description/meshes/visual/soft_finger.stl" scale="0.001 0.001 0.001"/>
         </geometry>
-        <material name="orange" />
+        <material name="${tf_prefix}orange" />
       </visual>
     <!--

Commit message: add configurable origin

File: urdf/diy_gripper_macro.urdf.xacro (robot description, xacro)
@@ -9,4 +9,5 @@
     <xacro:materials tf_prefix="${tf_prefix}"/>
       <joint name="${tf_prefix}gripper_to_parent" type="fixed">
+        <origin "${*origin}"/>
         <parent link="${parent}"/>
         <child link="${tf_prefix}base_link"/>

Commit message: modified origin

File: urdf/diy_gripper_macro.urdf.xacro (robot description, xacro)
@@ -9,5 +9,5 @@
     <xacro:materials tf_prefix="${tf_prefix}"/>
       <joint name="${tf_prefix}gripper_to_parent" type="fixed">
-        <origin "${*origin}"/>
+        <origin "${origin}"/>
         <parent link="${parent}"/>
         <child link="${tf_prefix}base_link"/>

Commit message: changed origin

File: urdf/diy_gripper_macro.urdf.xacro (robot description, xacro)
@@ -9,5 +9,5 @@
     <xacro:materials tf_prefix="${tf_prefix}"/>
       <joint name="${tf_prefix}gripper_to_parent" type="fixed">
-        <origin "${origin}"/>
+        <origin xyz="0 0 0.095" rpy="0 0 0"/>
         <parent link="${parent}"/>
         <child link="${tf_prefix}base_link"/>

Commit message: modified origin

File: urdf/diy_gripper_macro.urdf.xacro (robot description, xacro)
@@ -9,5 +9,4 @@
     <xacro:materials tf_prefix="${tf_prefix}"/>
       <joint name="${tf_prefix}gripper_to_parent" type="fixed">
-        <origin xyz="0 0 0.095" rpy="0 0 0"/>
         <parent link="${parent}"/>
         <child link="${tf_prefix}base_link"/>

Commit message: add collision mesh and delete transmission.urdf

File: urdf/diy_gripper_macro.urdf.xacro (robot description, xacro)
@@ -20,12 +20,10 @@
         <material name="${tf_prefix}grey" />
       </visual>
-    <!--
       <collision>
         <origin xyz="0 0 0" rpy="0 0 0" />
         <geometry>
-          <mesh filename="$(find diy_soft_gripper_description)/meshes/collision/base_link.stl" />
+          <mesh filename="$(find diy_soft_gripper_description)/meshes/collision/tool.stl" />
         </geometry>
       </collision>
-    -->
     </link>
     <joint name="${tf_prefix}right_joint" type="fixed">
@@ -43,12 +41,4 @@
         <material name="${tf_prefix}orange" />
       </visual>
-    <!--
-      <collision>
-        <origin xyz="0 0 0" rpy="0 0 0" />
-        <geometry>
-          <mesh filename="$(find diy_soft_gripper_description)/meshes/collision/soft_finger.stl" />
-        </geometry>
-      </collision>
-    -->
     </link>
     <joint name="${tf_prefix}left_joint" type="fixed">
@@ -66,14 +56,5 @@
         <material name="${tf_prefix}orange" />
       </visual>
-    <!--
-      <collision>
-        <origin xyz="0 0 0" rpy="0 0 0" />
-        <geometry>
-          <mesh filename="$(find diy_soft_gripper_description)/meshes/collision/soft_finger.stl" />
-        </geometry>
-      </collision>
-    -->
     </link>
   </xacro:macro>
-<!--<xacro:robotiq_arg2f_transmission tf_prefix="${tf_prefix}"/>, currently not used, because gripper is force-controlled without using ros2_control-->
 </robot>

Commit message: changed collision load path

File: urdf/diy_gripper_macro.urdf.xacro (robot description, xacro)
@@ -23,5 +23,5 @@
         <origin xyz="0 0 0" rpy="0 0 0" />
         <geometry>
-          <mesh filename="$(find diy_soft_gripper_description)/meshes/collision/tool.stl" />
+          <mesh filename="package://diy_soft_gripper_description/meshes/collision/tool.stl" />
         </geometry>
       </collision>

Commit message: scaled collision mesh impoort

File: urdf/diy_gripper_macro.urdf.xacro (robot description, xacro)
@@ -23,5 +23,5 @@
         <origin xyz="0 0 0" rpy="0 0 0" />
         <geometry>
-          <mesh filename="package://diy_soft_gripper_description/meshes/collision/tool.stl" />
+          <mesh filename="package://diy_soft_gripper_description/meshes/collision/tool.stl" scale="0.001 0.001 0.001"/>
         </geometry>
       </collision>

Commit message: changed collosion color and position

File: urdf/diy_gripper_macro.urdf.xacro (robot description, xacro)
@@ -21,8 +21,9 @@
       </visual>
       <collision>
-        <origin xyz="0 0 0" rpy="0 0 0" />
+        <origin xyz="0 0 0.027" rpy="0 0 0" />
         <geometry>
           <mesh filename="package://diy_soft_gripper_description/meshes/collision/tool.stl" scale="0.001 0.001 0.001"/>
         </geometry>
+        <material name="${tf_prefix}red" />
       </collision>
     </link>

Commit message: edited collision meshes

File: urdf/diy_gripper_macro.urdf.xacro (robot description, xacro)
@@ -21,5 +21,5 @@
       </visual>
       <collision>
-        <origin xyz="0 0 0.027" rpy="0 0 0" />
+        <origin xyz="0 0 0" rpy="0 0 0" />
         <geometry>
           <mesh filename="package://diy_soft_gripper_description/meshes/collision/tool.stl" scale="0.001 0.001 0.001"/>

Commit message: replaced collision mesh

File: urdf/diy_gripper_macro.urdf.xacro (robot description, xacro)
@@ -21,5 +21,5 @@
       </visual>
       <collision>
-        <origin xyz="0 0 0" rpy="0 0 0" />
+        <origin xyz="0 0 0.028" rpy="0 0 0" />
         <geometry>
           <mesh filename="package://diy_soft_gripper_description/meshes/collision/tool.stl" scale="0.001 0.001 0.001"/>

Commit message: moved the tcp link definition from model to macro urdf that it is also acessable in the full_cell_description

File: urdf/diy_gripper_macro.urdf.xacro (robot description, xacro)
@@ -59,3 +59,10 @@
     </link>
   </xacro:macro>
+   <!--add a TCP Link for convenience, show TCP reference set in rviz-->
+    <joint name="tcp_joint" type="fixed">
+        <origin xyz="0 0 0.08" rpy="0 0 0"/>
+        <parent link="$(arg tf_prefix)base_link"/>
+        <child link="$(arg tf_prefix)tcp_link"/>
+    </joint>
+    <link name="$(arg tf_prefix)tcp_link"/>
 </robot>

File: urdf/diy_gripper_model.urdf.xacro (robot description, xacro)
@@ -8,10 +8,3 @@
         <origin xyz="0 0 0" rpy="0 0 0"/>
     </xacro:diy_soft_gripper>
-    <!--add a TCP Link for convenience, show TCP reference set in rviz-->
-    <joint name="tcp_joint" type="fixed">
-        <origin xyz="0 0 0.08" rpy="0 0 0"/>
-        <parent link="$(arg tf_prefix)base_link"/>
-        <child link="$(arg tf_prefix)tcp_link"/>
-    </joint>
-    <link name="$(arg tf_prefix)tcp_link"/>
 </robot>

Commit message: changed tf_prefix from argument to parameter

File: urdf/diy_gripper_macro.urdf.xacro (robot description, xacro)
@@ -62,7 +62,7 @@
     <joint name="tcp_joint" type="fixed">
         <origin xyz="0 0 0.08" rpy="0 0 0"/>
-        <parent link="$(arg tf_prefix)base_link"/>
-        <child link="$(arg tf_prefix)tcp_link"/>
+        <parent link="${tf_prefix}base_link"/>
+        <child link="${tf_prefix}tcp_link"/>
     </joint>
-    <link name="$(arg tf_prefix)tcp_link"/>
+    <link name="${tf_prefix}tcp_link"/>
 </robot>

Commit message: solved tf_prefix param error

File: urdf/diy_gripper_macro.urdf.xacro (robot description, xacro)
@@ -58,7 +58,6 @@
       </visual>
     </link>
-  </xacro:macro>
-   <!--add a TCP Link for convenience, show TCP reference set in rviz-->
-    <joint name="tcp_joint" type="fixed">
+    <!--add a TCP Link for convenience, show TCP reference set in rviz-->
+    <joint name="${tf_prefix}tcp_joint" type="fixed">
         <origin xyz="0 0 0.08" rpy="0 0 0"/>
         <parent link="${tf_prefix}base_link"/>
@@ -66,3 +65,4 @@
     </joint>
     <link name="${tf_prefix}tcp_link"/>
+  </xacro:macro>
 </robot>

Commit message: delete build install and log and do some commits in urdf

File: urdf/diy_gripper_macro.urdf.xacro (robot description, xacro)
@@ -1,6 +1,4 @@
 <?xml version="1.0"?>
 <robot xmlns:xacro="http://ros.org/wiki/xacro">
-<!--include the transmissions macro , will not be used in this case but interesting when controlling the gripper via ros2_control position interface-->
-  <!--<xacro:include filename="$(find diy_soft_gripper_description)/urdf/diy_gripper_transmissions.urdf.xacro" /> -->
 <!--include the material/ colors macro-->
   <xacro:include filename="$(find diy_soft_gripper_description)/urdf/materials.urdf.xacro" />
@@ -8,5 +6,5 @@
   <xacro:macro name="diy_soft_gripper" params="tf_prefix parent *origin">
     <xacro:materials tf_prefix="${tf_prefix}"/>
-      <joint name="${tf_prefix}gripper_to_parent" type="fixed">
+    <joint name="${tf_prefix}gripper_to_parent" type="fixed">
         <parent link="${parent}"/>
         <child link="${tf_prefix}base_link"/>
